File: pcb/boes_sensor.kicad_pcb (KiCad board)
At the start: 2 copper layers, 41.1 x 18.3 mm, 13 parts, among them U1 LM358, Y1 Piezo

Commit message: Use teardrop pads for sensor PCB
Parts:
- renumbered C2 to C1, C1 to C2, R4 to R3, R3 to R4, TP3 to TP1, TP4 to TP2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

Commit message: Add decoupling to sensor VCC rail
Parts:
- added C3: 1u, Capacitor_SMD:C_0603_1608Metric, F.Cu at (142.7, 106.2)
- added C4: 100n, Capacitor_SMD:C_0603_1608Metric, F.Cu at (144.3, 106.2)
Routing:
- net VCC: track 10.2 -> 11.0 mm
