File: pcb/boes.kicad_sch (KiCad schematic)
At the start: 20 parts

Commit message: Separate main board from sensor boards
Parts:
- added RV?: Sens_Judge, symbol Device:R_Potentiometer
- added RV?: Sens_Participant, symbol Device:R_Potentiometer
Connections:
- new net Sens_Judge: RV?.2
- new net Sens_Participant: RV?.2
Changed lines of the file:
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@@
+    )
+  )
+  (global_label "Sens_Judge" (shape input) (at 220.98 85.09 180) (fields_autoplaced)
+    (effects (font (size 1.27 1.27)) (justify right))
+    (property "Intersheet References" "${INTERSHEET_REFS}" (id 0) (at 207.6207 85.0106 0)
+      (effects (font (size 1.27 1.27)) (justify right) hide)
     )
   )
@@
     (effects (font (size 1.27 1.27)) (justify right))
     (property "Intersheet References" "${INTERSHEET_REFS}" (id 0) (at 160.2074 98.9806 0)
+      (effects (font (size 1.27 1.27)) (justify right) hide)
+    )
+  )
+  (global_label "Sens_Participant" (shape input) (at 220.98 99.06 180) (fields_autoplaced)
+    (effects (font (size 1.27 1.27)) (justify right))
+    (property "Intersheet References" "${INTERSHEET_REFS}" (id 0) (at 202.7221 98.9806 0)
       (effects (font (size 1.27 1.27)) (justify right) hide)
     )
@@
     )
     (pin "1")
+  )
+  (symbol (lib_id "Device:R_Potentiometer") (at 224.79 85.09 0) (mirror y) (unit 1)
+    (in_bom yes) (on_board yes) (fields_autoplaced)
+    (property "Reference" "RV?" (id 0) (at 226.568 84.1815 0)
+      (effects (font (size 1.27 1.27)) (justify right))
+    )
+    (property "Value" "Sens_Judge" (id 1) (at 226.568 86.9566 0)
+      (effects (font (size 1.27 1.27)) (justify right))
+    )
+    (property "Footprint" "" (id 2) (at 224.79 85.09 0)
+      (effects (font (size 1.27 1.27)) hide)
+    )
+    (property "Datasheet" "~" (id 3) (at 224.79 85.09 0)
+      (effects (font (size 1.27 1.27)) hide)
+    )
+    (pin "1")
+    (pin "2")
+    (pin "3")
   )
   (symbol (lib_id "Connector_Generic:Conn_01x03") (at 259.08 137.16 0) (unit 1)
@@
     (pin "2")
   )
+  (symbol (lib_id "Device:R_Potentiometer") (at 224.79 99.06 0) (mirror y) (unit 1)
+    (in_bom yes) (on_board yes) (fields_autoplaced)
+    (property "Reference" "RV?" (id 0) (at 226.568 98.1515 0)
+      (effects (font (size 1.27 1.27)) (justify right))
+    )
+    (property "Value" "Sens_Participant" (id 1) (at 226.568 100.9266 0)
+      (effects (font (size 1.27 1.27)) (justify right))
+    )
+    (property "Footprint" "" (id 2) (at 224.79 99.06 0)
+      (effects (font (size 1.27 1.27)) hide)
+    )
+    (property "Datasheet" "~" (id 3) (at 224.79 99.06 0)
+      (effects (font (size 1.27 1.27)) hide)
+    )
+    (pin "1")
+    (pin "2")
+    (pin "3")
+  )
   (symbol (lib_id "Diode:BAV99") (at 180.975 153.67 0) (unit 1)
     (in_bom yes) (on_board yes) (fields_autoplaced)
@@
     (pin "2")
     (pin "3")
-    (pin "5")
-    (pin "6")
-    (pin "7")
-    (pin "4")
-    (pin "8")
   )
   (sheet_instances
@@
       (reference "R?") (unit 1) (value "R") (footprint "")
     )
+    (path "/6cf57bed-2ba3-4e7f-94fe-42c6a93dee9a"
+      (reference "RV?") (unit 1) (value "Sens_Judge") (footprint "")
+    )
+    (path "/e3c978d7-e028-4704-9fee-d84a5f934236"
+      (reference "RV?") (unit 1) (value "Sens_Participant") (footprint "")
+    )
     (path "/0415c2e6-5728-4890-b5cd-2d863d83a975"

Commit message: Almost finished main board
Parts:
- removed C?: 100n, symbol Device:C
- removed D?: 1N4148, symbol Device:D
- removed D?: BAV99, Package_TO_SOT_SMD:SOT-23, symbol Diode:BAV99
- removed J?: USB_C_Receptacle_USB2.0, symbol Connector:USB_C_Receptacle_USB2.0
- removed LS?: Speaker, symbol Device:Speaker
- removed R? (x2): R, symbol Device:R
- removed R?: 100k, symbol Device:R
- removed RV?: Sens_Participant, symbol Device:R_Potentiometer
- removed U?: LM358, symbol Amplifier_Operational:LM358
- added BZ1: Buzzer, symbol Device:Buzzer
- added H1, H2, H3, H4: MountingHole, MountingHole:MountingHole_3.2mm_M3, symbol Mechanical:MountingHole
- added J1: SW_A, Connector_JST:JST_XH_B2B-XH-A_1x02_P2.50mm_Vertical, symbol Connector_Generic:Conn_01x02
- added J2: SW_B, Connector_JST:JST_XH_B2B-XH-A_1x02_P2.50mm_Vertical, symbol Connector_Generic:Conn_01x02
- added J3: SW_C, Connector_JST:JST_XH_B2B-XH-A_1x02_P2.50mm_Vertical, symbol Connector_Generic:Conn_01x02
- added J4: Pot_J, Connector_JST:JST_XH_B3B-XH-A_1x03_P2.50mm_Vertical, symbol Connector_Generic:Conn_01x03
- added J5: Pot_P, Connector_JST:JST_XH_B3B-XH-A_1x03_P2.50mm_Vertical, symbol Connector_Generic:Conn_01x03
- added J8: Buzzer, Connector_JST:JST_XH_B2B-XH-A_1x02_P2.50mm_Vertical, symbol Connector_Generic:Conn_01x02
- added P1: SW_A, symbol Connector_Generic:Conn_01x02
- added P2: SW_B, symbol Connector_Generic:Conn_01x02
- added P3: SW_C, symbol Connector_Generic:Conn_01x02
- added P4: Pot_J, symbol Connector_Generic:Conn_01x03
- added P5: Pot_P, symbol Connector_Generic:Conn_01x03
- added P8: Buzzer, symbol Connector_Generic:Conn_01x02
- added RV2: Pot_P, symbol Device:R_Potentiometer
- J10: renamed from J?; footprint (none) -> Connector_IDC:IDC-Header_2x08_P2.54mm_Vertical
- J6: renamed from J?; value Judge -> Sens_J; footprint (none) -> Connector_JST:JST_XH_B3B-XH-A_1x03_P2.50mm_Vertical
- J7: renamed from J?; value Participant -> Sens_P; footprint (none) -> Connector_JST:JST_XH_B3B-XH-A_1x03_P2.50mm_Vertical
- J9: renamed from J?; footprint (none) -> TerminalBlock_Phoenix:TerminalBlock_Phoenix_MKDS-1,5-2-5.08_1x02_P5.08mm_Horizontal
- Q1: renamed from Q?; footprint Package_TO_SOT_THT:TO-92_Inline -> Package_TO_SOT_SMD:SOT-23
- R1: renamed from R?; value R -> 10k; footprint (none) -> Resistor_SMD:R_0603_1608Metric
- R2: renamed from R?; footprint (none) -> Resistor_SMD:R_0603_1608Metric
- RV1: renamed from RV?; value Sens_Judge -> Pot_J
- gave numbers to parts that had none: 4
Connections:
- net +5V: now also U1.40 (VBUS), J8.1 (Pin_1)
- net A: now also U1.10 (GPIO7)
- net B: now also U1.11 (GPIO8)
- net B1: now also U1.4 (GPIO2)
- net B2: now also U1.7 (GPIO5)
- net Buzzer: now also U1.21 (GPIO16)
- net C: now also U1.12 (GPIO9)
- net CLK: now also U1.15 (GPIO11)
- net D: now also U1.14 (GPIO10)
- net E: now also U1.9 (GPIO6)
- net G1: now also U1.2 (GPIO1)
- net G2: now also U1.6 (GPIO4)
- net GND: now also J6.3 (Pin_3), J7.3 (Pin_3), J1.2 (Pin_2), J2.2 (Pin_2), J3.2 (Pin_2), J4.3 (Pin_3), J5.3 (Pin_3); no longer SW1.2, SW2.2, SW3.2
- net Latch: now also U1.16 (GPIO12)
- net OE: now also U1.17 (GPIO13)
- net R1: now also U1.1 (GPIO0)
- net R2: now also U1.5 (GPIO3)
- net Reset: now also U1.22 (GPIO17), J3.1 (Pin_1); no longer SW3.1
- net Start: now also U1.25 (GPIO19), J1.1 (Pin_1); no longer SW1.1
- net Stop: now also U1.24 (GPIO18), J2.1 (Pin_1); no longer SW2.1
- net at RV1.1: now also P4.1 (Pin_1)
- net at RV1.3: now also P4.3 (Pin_3)
- net +3V3: now reaches J6.1 (Pin_1)
- net +3V3: now also J7.1 (Pin_1), U1.36 (3V3), J4.1 (Pin_1), J5.1 (Pin_1)
- net Sens_J: now reaches J6.2 (Pin_2)
- net Sens_J: now also U1.32 (GPIO27_ADC1)
- net at R2.1: now also J8.2 (Pin_2)
- net Sens_P: now reaches U1.31 (GPIO26_ADC0)
- net Sens_P: now also J7.2 (Pin_2)
- net Sens_Judge: no longer names the net of RV1.2
- net Sens_Judge: now also P4.2 (Pin_2)
- new net: P2.1 (Pin_1), SW2.1
- new net: P2.2 (Pin_2), SW2.2
- new net: P1.1 (Pin_1), SW1.1
- new net: P1.2 (Pin_2), SW1.2
- new net: P5.1 (Pin_1), RV2.1
- new net: P5.2 (Pin_2), RV2.2
- new net: P5.3 (Pin_3), RV2.3
- new net: P3.1 (Pin_1), SW3.1
- new net: P3.2 (Pin_2), SW3.2
- new net: BZ1.1 (-), P8.1 (Pin_1)
- new net: BZ1.2 (+), P8.2 (Pin_2)
- new net Pot_J: J4.2 (Pin_2)
- new net Pot_P: J5.2 (Pin_2)
- no-connect marks 0 -> 2
Other:
- note added: "Control buttons"
- note added: "Sensitivity potentiometers"
- note added: "Sensor connectors"
- note removed: "Can amplifiers / filters be at main board? Needs testing!"
- note removed: "Is a peak detector needed? Only if the ADC conversion might miss the peak/pulse."
- note removed: "Should it be possible to change volume?"
- note removed: "Transient limit to ±0,7V"
- moved on the sheet: J6, J7, J9, Q1, R1, R2, RV1, SW1, SW2, SW3, U1

Commit message: Slim main PCB
Parts:
- removed J5: Pot_P, Connector_JST:JST_XH_B3B-XH-A_1x03_P2.50mm_Vertical, symbol Connector_Generic:Conn_01x03
- removed P5: Pot_P, symbol Connector_Generic:Conn_01x03
- removed RV2: Pot_P, symbol Device:R_Potentiometer
- RV1: value Pot_J -> 10k
Connections:
- net Pot_J is gone; now on net Pot: J4.2 (Pin_2)
- net A: now also U1.12 (GPIO9); no longer U1.10 (GPIO7)
- net B: now also U1.14 (GPIO10); no longer U1.11 (GPIO8)
- net B1: now also U1.5 (GPIO3); no longer U1.4 (GPIO2)
- net B2: now also U1.10 (GPIO7); no longer U1.7 (GPIO5)
- net C: now also U1.15 (GPIO11); no longer U1.12 (GPIO9)
- net CLK: now also U1.20 (GPIO15); no longer U1.15 (GPIO11)
- net D: now also U1.16 (GPIO12); no longer U1.14 (GPIO10)
- net E: now also U1.11 (GPIO8); no longer U1.9 (GPIO6)
- net G1: now also U1.7 (GPIO5); no longer U1.2 (GPIO1)
- net G2: now also U1.9 (GPIO6); no longer U1.6 (GPIO4)
- net Latch: now also U1.17 (GPIO13); no longer U1.16 (GPIO12)
- net OE: now also U1.19 (GPIO14); no longer U1.17 (GPIO13)
- net R1: now also U1.6 (GPIO4); no longer U1.1 (GPIO0)
- net R2: now also U1.4 (GPIO2); no longer U1.5 (GPIO3)
- net Start: now also U1.29 (GPIO22); no longer U1.25 (GPIO19)
- net Stop: now also U1.27 (GPIO21); no longer U1.24 (GPIO18)
- net Pot: now reaches U1.34 (GPIO28_ADC2)
- no-connect marks 2 -> 9
