File: pcb/boes.kicad_sch (KiCad schematic)
At the start: 27 parts, among them J1 SW_A, J10 HUB75 Display ctrl, J2 SW_B, J3 SW_C, J4 Pot_J, J6 Sens_J, J7 Sens_P, J8 Buzzer, J9 Display power, P1 SW_A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

Commit message: Repurpose screw terminal as input
Parts:
- added D1: D_Schottky, Diode_SMD:D_SMA-SMB_Universal_Handsoldering, symbol Device:D_Schottky
- J9: value Display power -> +5V External
Connections:
- net VCC: now reaches U1.39 (VSYS)
- net VCC: now also J8.1 (Pin_1), D1.1 (K)
- removed net +5V: J8.1 (Pin_1), J9.1 (Pin_1), U1.40 (VBUS)
- new net: D1.2 (A), J9.1 (Pin_1)
- no-connect marks 9 -> 11
Other:
- note removed: "Max 2.5A"
- moved on the sheet: J9
