File: pcb/boes_usb-c.kicad_sch (KiCad schematic)
At the start: 9 parts, among them J1 USB_C_Receptacle_USB2.0

Commit message: Improve strain relief
Parts:
- TP1, TP4: footprint Connector_Wire:SolderWire-0.1sqmm_1x01_D0.4mm_OD1mm_Relief -> Connector_Wire:SolderWire-0.5sqmm_1x01_D0.9mm_OD2.1mm_Relief
Changed lines of the file:
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@@
       (effects (font (size 1.27 1.27)) (justify left))
     )
-    (property "Footprint" "Connector_Wire:SolderWire-0.1sqmm_1x01_D0.4mm_OD1mm_Relief" (at 123.19 55.88 0)
+    (property "Footprint" "Connector_Wire:SolderWire-0.5sqmm_1x01_D0.9mm_OD2.1mm_Relief" (at 123.19 55.88 0)
       (effects (font (size 1.27 1.27)) hide)
     )
@@
       (effects (font (size 1.27 1.27)) (justify left))
     )
-    (property "Footprint" "Connector_Wire:SolderWire-0.1sqmm_1x01_D0.4mm_OD1mm_Relief" (at 123.19 80.01 0)
+    (property "Footprint" "Connector_Wire:SolderWire-0.5sqmm_1x01_D0.9mm_OD2.1mm_Relief" (at 123.19 80.01 0)
       (effects (font (size 1.27 1.27)) hide)
     )
